File: sensors/bee_counter/counter_shield.brd (EAGLE design)
At the start: 100 x 80 mm, 34 parts, among them IC1 74LS595N, IC2 74LS595N

Commit message: logo
Parts:
- removed IC1, IC2: 74LS595N, 01_SparkFun:DIL16
- added JP1: M25PTH_LONGPADS, SparkFun-Connectors:1X25_LONGPAD
- moved U$1 2.00 mm to (78.7, 75.7)
- moved U$17 2.00 mm to (63.5, 75.7)
- moved U$9 2.00 mm to (71.1, 75.7)
Connections:
- net GND: now also JP1.2; no longer IC1.8, IC2.8
- net VCC: now also JP1.1; no longer IC1.16, IC2.16
Changed lines of the file:
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@@
 <setting verticaltext="up"/>
 </settings>
-<grid distance="0.05" unitdist="inch" unit="inch" style="lines" multiple="1" display="yes" altdistance="0.005" altunitdist="inch" altunit="inch"/>
+<grid distance="1" unitdist="mm" unit="mm" style="lines" multiple="1" display="yes" altdistance="0.005" altunitdist="inch" altunit="inch"/>
 <layers>
 <layer number="1" name="Top" color="4" fill="1" visible="yes" active="yes"/>
@@
 <layer number="144" name="Drill_legend" color="7" fill="1" visible="no" active="yes"/>
 <layer number="151" name="HeatSink" color="7" fill="1" visible="no" active="yes"/>
+<layer number="199" name="Contour" color="7" fill="1" visible="yes" active="yes"/>
 <layer number="200" name="200bmp" color="1" fill="10" visible="no" active="yes"/>
 <layer number="201" name="201bmp" color="2" fill="10" visible="no" active="yes"/>
@@
 </autorouter>
 <elements>
-<element name="IC1" library="01_SparkFun" package="DIL16" value="74LS595N" x="74.93" y="11.43"/>
-<element name="IC2" library="01_SparkFun" package="DIL16" value="74LS595N" x="74.93" y="24.13"/>
-<element name="U$1" library="SparkFun-Sensors" package="QRE1113" value="QRE1113" x="78.74" y="73.66"/>
+<element name="U$1" library="SparkFun-Sensors" package="QRE1113" value="QRE1113" x="78.74" y="75.66"/>
 <element name="U$2" library="SparkFun-Sensors" package="QRE1113" value="QRE1113" x="78.74" y="68.58"/>
 <element name="U$3" library="SparkFun-Sensors" package="QRE1113" value="QRE1113" x="78.74" y="63.5"/>
@@
 <element name="U$7" library="SparkFun-Sensors" package="QRE1113" value="QRE1113" x="78.74" y="43.18"/>
 <element name="U$8" library="SparkFun-Sensors" package="QRE1113" value="QRE1113" x="78.74" y="38.1"/>
-<element name="U$9" library="SparkFun-Sensors" package="QRE1113" value="QRE1113" x="71.12" y="73.66"/>
+<element name="U$9" library="SparkFun-Sensors" package="QRE1113" value="QRE1113" x="71.12" y="75.66"/>
 <element name="U$10" library="SparkFun-Sensors" package="QRE1113" value="QRE1113" x="71.12" y="68.58"/>
 <element name="U$11" library="SparkFun-Sensors" package="QRE1113" value="QRE1113" x="71.12" y="63.5"/>
@@
 <element name="U$15" library="SparkFun-Sensors" package="QRE1113" value="QRE1113" x="71.12" y="43.18"/>
 <element name="U$16" library="SparkFun-Sensors" package="QRE1113" value="QRE1113" x="71.12" y="38.1"/>
-<element name="U$17" library="SparkFun-Sensors" package="QRE1113" value="QRE1113" x="63.5" y="73.66"/>
+<element name="U$17" library="SparkFun-Sensors" package="QRE1113" value="QRE1113" x="63.5" y="75.66"/>
 <element name="U$18" library="SparkFun-Sensors" package="QRE1113" value="QRE1113" x="63.5" y="68.58"/>
 <element name="U$19" library="SparkFun-Sensors" package="QRE1113" value="QRE1113" x="63.5" y="63.5"/>
@@
 <element name="R7" library="01_ng" package="1206" value="33" x="86.36" y="43.18"/>
 <element name="R8" library="01_ng" package="1206" value="33" x="86.36" y="38.1"/>
+<element name="JP1" library="SparkFun-Connectors" package="1X25_LONGPAD" value="M25PTH_LONGPADS" x="96.52" y="76.2" rot="R270"/>
 </elements>
 <signals>
 <signal name="GND">
-<contactref element="IC1" pad="8"/>
-<contactref element="IC2" pad="8"/>
 <contactref element="R1" pad="2"/>
 <contactref element="R2" pad="2"/>
@@
 <contactref element="R7" pad="2"/>
 <contactref element="R8" pad="2"/>
-<wire x1="87.782" y1="68.58" x2="87.782" y2="73.66" width="0" layer="19" extent="1-1"/>
+<contactref element="JP1" pad="2"/>
+<wire x1="87.782" y1="68.58" x2="96.52" y2="73.66" width="0" layer="19" extent="1-1"/>
+<wire x1="87.782" y1="73.66" x2="87.782" y2="68.58" width="0" layer="19" extent="1-1"/>
 <wire x1="87.782" y1="63.5" x2="87.782" y2="68.58" width="0" layer="19" extent="1-1"/>
 <wire x1="87.782" y1="58.42" x2="87.782" y2="63.5" width="0" layer="19" extent="1-1"/>
@@
 <wire x1="87.782" y1="43.18" x2="87.782" y2="48.26" width="0" layer="19" extent="1-1"/>
 <wire x1="87.782" y1="38.1" x2="87.782" y2="43.18" width="0" layer="19" extent="1-1"/>
-<wire x1="83.82" y1="20.32" x2="87.782" y2="38.1" width="0" layer="19" extent="1-1"/>
-<wire x1="83.82" y1="7.62" x2="83.82" y2="20.32" width="0" layer="19" extent="1-1"/>
 </signal>
 <signal name="VCC">
-<contactref element="IC1" pad="16"/>
-<contactref element="IC2" pad="16"/>
 <contactref element="U$17" pad="1"/>
 <contactref element="U$18" pad="1"/>
@@
 <contactref element="U$7" pad="3"/>
 <contactref element="U$8" pad="3"/>
-<wire x1="80.54" y1="69.48" x2="80.54" y2="74.56" width="0" layer="19" extent="1-1"/>
+<contactref element="JP1" pad="1"/>
+<wire x1="80.54" y1="76.56" x2="80.54" y2="69.48" width="0" layer="19" extent="1-1"/>
 <wire x1="80.54" y1="64.4" x2="80.54" y2="69.48" width="0" layer="19" extent="1-1"/>
 <wire x1="80.54" y1="59.32" x2="80.54" y2="64.4" width="0" layer="19" extent="1-1"/>
@@
 <wire x1="80.54" y1="44.08" x2="80.54" y2="49.16" width="0" layer="19" extent="1-1"/>
 <wire x1="80.54" y1="39" x2="80.54" y2="44.08" width="0" layer="19" extent="1-1"/>
-<wire x1="72.92" y1="74.56" x2="80.54" y2="74.56" width="0" layer="19" extent="1-1"/>
-<wire x1="72.92" y1="69.48" x2="72.92" y2="74.56" width="0" layer="19" extent="1-1"/>
+<wire x1="72.92" y1="69.48" x2="72.92" y2="76.56" width="0" layer="19" extent="1-1"/>
 <wire x1="72.92" y1="64.4" x2="72.92" y2="69.48" width="0" layer="19" extent="1-1"/>
 <wire x1="72.92" y1="59.32" x2="72.92" y2="64.4" width="0" layer="19" extent="1-1"/>
@@
 <wire x1="72.92" y1="44.08" x2="72.92" y2="49.16" width="0" layer="19" extent="1-1"/>
 <wire x1="72.92" y1="39" x2="72.92" y2="44.08" width="0" layer="19" extent="1-1"/>
-<wire x1="65.3" y1="74.56" x2="72.92" y2="74.56" width="0" layer="19" extent="1-1"/>
-<wire x1="61.7" y1="72.76" x2="65.3" y2="74.56" width="0" layer="19" extent="1-1"/>
-<wire x1="65.3" y1="69.48" x2="61.7" y2="72.76" width="0" layer="19" extent="1-1"/>
+<wire x1="61.7" y1="74.76" x2="65.3" y2="76.56" width="0" layer="19" extent="1-1"/>
+<wire x1="65.3" y1="69.48" x2="61.7" y2="74.76" width="0" layer="19" extent="1-1"/>
 <wire x1="61.7" y1="67.68" x2="65.3" y2="69.48" width="0" layer="19" extent="1-1"/>
 <wire x1="65.3" y1="64.4" x2="61.7" y2="67.68" width="0" layer="19" extent="1-1"/>
@@
 <wire x1="65.3" y1="39" x2="61.7" y2="42.28" width="0" layer="19" extent="1-1"/>
 <wire x1="61.7" y1="37.2" x2="65.3" y2="39" width="0" layer="19" extent="1-1"/>
-<wire x1="66.04" y1="27.94" x2="61.7" y2="37.2" width="0" layer="19" extent="1-1"/>
-<wire x1="66.04" y1="15.24" x2="66.04" y2="27.94" width="0" layer="19" extent="1-1"/>
+<wire x1="80.54" y1="69.48" x2="96.52" y2="76.2" width="0" layer="19" extent="1-1"/>
+<wire x1="65.3" y1="76.56" x2="72.92" y2="76.56" width="0" layer="19" extent="1-1"/>
+<wire x1="72.92" y1="76.56" x2="80.54" y2="76.56" width="0" layer="19" extent="1-1"/>
 </signal>
 <signal name="N$1">
 <contactref element="U$17" pad="2"/>
 <contactref element="U$9" pad="1"/>
-<wire x1="65.3" y1="72.76" x2="69.32" y2="72.76" width="0" layer="19" extent="1-1"/>
+<wire x1="65.3" y1="74.76" x2="69.32" y2="74.76" width="0" layer="19" extent="1-1"/>
 </signal>
 <signal name="N$2">
 <contactref element="U$9" pad="2"/>
 <contactref element="U$1" pad="1"/>
-<wire x1="72.92" y1="72.76" x2="76.94" y2="72.76" width="0" layer="19" extent="1-1"/>
+<wire x1="72.92" y1="74.76" x2="76.94" y2="74.76" width="0" layer="19" extent="1-1"/>
 </signal>
 <signal name="N$3">
@@
 <contactref element="R1" pad="1"/>
 <contactref element="U$1" pad="2"/>
-<wire x1="80.54" y1="72.76" x2="84.938" y2="73.66" width="0" layer="19" extent="1-1"/>
+<wire x1="80.54" y1="74.76" x2="84.938" y2="73.66" width="0" layer="19" extent="1-1"/>
 </signal>
 <signal name="N$25">

Commit message: laser stuff
Parts:
- removed JP1: M25PTH_LONGPADS, SparkFun-Connectors:1X25_LONGPAD
- removed R1, R2, R3, R4, R5, R6, R7: 33, 01_ng:1206
- removed U$1, U$10, U$11, U$12, U$13, U$14, U$15, U$16, U$17, U$18, U$19, U$2, U$20, U$21, U$22, U$23, U$24, U$3, U$4, U$5, U$8: QRE1113, SparkFun-Sensors:QRE1113
- added R10, R11: 10k, 01_ng:1206
- R8: value 33 -> 100
- U$9: value QRE1113 -> M18_; device SparkFun-Sensors:QRE1113 -> SparkFun-Connectors:1X18
- moved U$9 86.9 mm to (4.81, 19.4), turned to 90 degrees
- moved U$7 72.6 mm to (9.73, 20.8)
- moved U$6 63.0 mm to (22.1, 20.6)
- moved R8 62.3 mm to (26.4, 21.2), turned to 90 degrees
Connections:
- removed net N$1: U$17.2, U$9.1
- removed net N$14: U$15.2, U$7.1
- removed net N$15: U$16.2, U$8.1
- removed net N$16: U$16.1, U$24.2
- removed net N$17: R8.1, U$8.2
- removed net N$18: R7.1, U$7.2
- removed net N$19: R6.1, U$6.2
- removed net N$2: U$1.1, U$9.2
- removed net N$20: R5.1, U$5.2
- removed net N$21: R4.1, U$4.2
- removed net N$22: R3.1, U$3.2
- removed net N$23: R2.1, U$2.2
- removed net N$24: R1.1, U$1.2
- removed net N$25: U$17.4
- removed net N$26: U$9.4
- removed net N$27: U$1.4
- removed net N$28: U$18.4
- removed net N$29: U$10.4
- removed net N$3: U$10.1, U$18.2
- removed net N$30: U$2.4
- removed net N$31: U$19.4
- removed net N$32: U$11.4
- removed net N$33: U$3.4
- removed net N$34: U$20.4
- removed net N$35: U$12.4
- removed net N$36: U$4.4
- removed net N$37: U$21.4
- removed net N$38: U$13.4
- removed net N$39: U$5.4
- removed net N$4: U$10.2, U$2.1
- removed net N$40: U$22.4
- removed net N$41: U$14.4
- removed net N$42: U$6.4
- removed net N$43: U$23.4
- removed net N$44: U$15.4
- removed net N$45: U$7.4
- removed net N$46: U$24.4
- removed net N$47: U$16.4
- removed net N$48: U$8.4
- removed net N$5: U$11.2, U$3.1
- removed net N$6: U$11.1, U$19.2
- removed net N$7: U$12.1, U$20.2
- removed net N$8: U$12.2, U$4.1
- removed net N$9: U$13.1, U$21.2
- net GND: now also U$6.4, U$7.4, U$9.2; no longer JP1.2, R1.2, R2.2, R3.2, R4.2, R5.2, R6.2, R7.2
- net N$10: now also R8.1, U$6.2; no longer U$13.2, U$5.1
- net N$11: now also U$7.2; no longer U$14.2
- net N$12: now also R10.1, U$7.3, U$9.3; no longer U$14.1, U$22.2
- net N$13: now also R11.1, U$6.3, U$9.4; no longer U$15.1, U$23.2
- net VCC: now also R10.2, R11.2, U$7.1, U$9.1; no longer JP1.1, U$1.3, U$10.3, U$11.3, U$12.3, U$13.3, U$14.3, U$15.3, U$16.3, U$17.1, U$17.3, U$18.1, U$18.3, U$19.1, U$19.3, U$2.3, U$20.1, U$20.3, U$21.1, U$21.3, U$22.1, U$22.3, U$23.1, U$23.3, U$24.1, U$24.3, U$3.3, U$4.3, U$5.3, U$6.3, U$7.3, U$8.3, U$9.3
Routing:
- net N$13: track 0.00 -> 33.0 mm
- net VCC: track 0.00 -> 28.7 mm
- net GND: track 0.00 -> 22.7 mm
- net N$12: track 0.00 -> 10.8 mm
- net N$11: track 0.00 -> 10.7 mm
- net N$10: track 0.00 -> 2.54 mm
Other:
- board size 100 x 80 mm -> 29.6 x 80.2 mm
